File: qds-cv-bypass-adapter.kicad_pcb (KiCad board)
At the start: 2 copper layers, 82.6 x 18.5 mm, 16 parts, among them J1 Conn_01x02, J2 Conn_02x05_Odd_Even, J3 Conn_01x02, J4 Conn_02x05_Odd_Even, SW1 SW_DPST, SW2 SW_DPST, SW3 SW_DPST, SW4 SW_DPST, SW5 SW_DPST, SW6 SW_DPST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

Commit message: 1a versão fabricada
Parts:
- removed the J1 at (127.6, 60.7)
- removed the J2 at (175.6, 61.2)
- removed the REF** at (117.9, 62.4)
- removed the REF** at (197.9, 62.5)
- removed the SW1 at (143.1, 62.5)
- removed the SW2 at (151.4, 62.5)
- removed the SW3 at (159.8, 62.5)
- removed the SW4 at (168.2, 62.5)
- moved SW1 0.91 mm to (143.5, 89.6)
- moved SW2 0.91 mm to (151.1, 89.6)
- moved SW3 0.91 mm to (158.8, 89.6)
- moved SW4 0.91 mm to (166.4, 89.6)
- moved J2 0.82 mm to (172.5, 85.1)
- moved J1 0.31 mm to (205.0, 89.3)
- moved REF** 0.31 mm to (134.9, 89.0)
- moved REF** 0.31 mm to (196.8, 89.0)
- renumbered J3 to J1, J4 to J2, SW5 to SW1, SW6 to SW2, SW7 to SW3, SW8 to SW4
Connections:
- J1 pad 1: Net-(J3-Pad1) -> Net-(SW1-Pad4)
- J1 pad 2: Net-(J3-Pad2) -> Net-(SW1-Pad1)
- SW1 pad 1: Net-(J3-Pad1) -> Net-(SW1-Pad1)
- SW1 pad 4: Net-(J3-Pad2) -> Net-(SW1-Pad4)
- SW2 pad 1: Net-(J3-Pad1) -> Net-(SW1-Pad1)
- SW2 pad 4: Net-(J3-Pad2) -> Net-(SW1-Pad4)
- SW3 pad 1: Net-(J3-Pad1) -> Net-(SW1-Pad1)
- SW3 pad 4: Net-(J3-Pad2) -> Net-(SW1-Pad4)
- SW4 pad 1: Net-(J3-Pad1) -> Net-(SW1-Pad1)
- SW4 pad 4: Net-(J3-Pad2) -> Net-(SW1-Pad4)
Routing:
- net Net-(J3-Pad2): track 86.2 -> 0.00 mm, vias 1 -> 0
- net Net-(J3-Pad1): track 83.2 -> 0.00 mm, vias 1 -> 0
- net Net-(SW1-Pad4): track 0.00 -> 81.4 mm, vias 0 -> 1
- net Net-(SW1-Pad1): track 0.00 -> 79.8 mm, vias 0 -> 1
- net Net-(J1-Pad1): track 49.7 -> 0.00 mm
- net Net-(J1-Pad2): track 44.8 -> 0.00 mm
- net Net-(J2-Pad7) (its old number): track 43.7 -> 0.00 mm
- net Net-(J2-Pad8) (its old number): track 43.6 -> 0.00 mm
- net Net-(J2-Pad6) (its old number): track 32.1 -> 0.00 mm
- net Net-(J2-Pad5) (its old number): track 31.8 -> 0.00 mm
- net Net-(J2-Pad4) (its old number): track 20.4 -> 0.00 mm
- net Net-(J2-Pad3) (its old number): track 20.3 -> 0.00 mm
- net Net-(J2-Pad2) (its old number): track 7.79 -> 0.00 mm
- net Net-(J2-Pad1) (its old number): track 7.79 -> 0.00 mm
- net Net-(J2-Pad4): track 20.6 -> 21.3 mm
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Other:
- board size 82.6 x 18.5 mm -> 82.6 x 19.6 mm
