File: qds-cv-bypass-adapter.kicad_sch (KiCad schematic)
At the start: 12 parts, among them J1 Conn_01x02, J2 Conn_02x05_Odd_Even, J3 Conn_01x02, J4 Conn_02x05_Odd_Even, SW1 SW_DPST, SW2 SW_DPST, SW3 SW_DPST, SW4 SW_DPST, SW5 SW_DPST, SW6 SW_DPST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

Commit message: 1a versão fabricada
Parts:
- removed J1: Conn_01x02, Connector_Phoenix_MC:PhoenixContact_MCV_1,5_2-G-3.81_1x02_P3.81mm_Vertical, symbol Connector_Generic:Conn_01x02
- removed J2: Conn_02x05_Odd_Even, qds-cv-bypass:SBH11PBPCD05STBK, symbol Connector_Generic:Conn_02x05_Odd_Even
- removed SW1, SW2, SW3, SW4: SW_DPST, qds-cv-bypass:204211STR, symbol Switch:SW_DIP_x02
- renumbered J3 to J1, J4 to J2, SW5 to SW1, SW6 to SW2, SW7 to SW3, SW8 to SW4
Connections:
- net at SW1.1, SW2.1, SW3.1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: now also J1.2 (Pin_2); no longer J1.1 (Pin_1)
- net at SW1.4, SW2.4, SW3.4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: now also J1.1 (Pin_1); no longer J1.2 (Pin_2)
Other:
- moved on the sheet: J1, J2, SW1, SW2, SW3, SW4
